Commit message: added lidar to the mollyBot, lidar is working

File: src/mollyBot/description/robot.urdf.xacro (robot description, xacro)
@@ -3,3 +3,4 @@
     <xacro:include filename="robot_core.xacro" />
     <xacro:include filename="gazebo_control.xacro" />
+    <xacro:include filename="lidar.xacro"/>
 </robot>

File: src/mollyBot/description/robot_core.xacro (robot description, xacro)
@@ -1,4 +1,8 @@
 <?xml version="1.0"?>
 <robot xmlns:xacro="http://www.ros.org/wiki/xacro" name="simple_bot">
+  <xacro:include filename="inertial_macros.xacro"/>
+  <material name="red">
+    <color rgba="1 0 0 1"/>
+  </material>
   <!-- Properties for easy modification -->
   <xacro:property name="wheel_radius" value="0.08" /> <!-- 3 inches / 2 -->
@@ -15,7 +19,7 @@
     <collision>
         <geometry>
-        <cylinder radius="${chassis_radius}" length="${chassis_height}"/>
+          <cylinder radius="${chassis_radius}" length="${chassis_height}"/>
         </geometry>
-      </collision>
+    </collision>
     <inertial>
       <origin xyz="0 0 0"/>
