Commit message: Added a chassis link so that inertia warning goes away for the base_link.

File: src/mollyBot/description/lidar.xacro (robot description, xacro)
@@ -2,5 +2,5 @@
 <robot xmlns:xacro="http://www.ros.org/wiki/xacro" >
     <joint name="laser_joint" type="fixed">
-        <parent link="base_link"/>
+        <parent link="chassis"/>
         <child link="laser_frame"/>
         <origin xyz="0.1 0 0.05" rpy="0 0 0"/>

File: src/mollyBot/description/robot_core.xacro (robot description, xacro)
@@ -12,4 +12,12 @@
   <!-- Base Link -->
   <link name="base_link">
+  </link>
+  <!-- Chassis Link -->
+  <joint name="chassis_joint" type="fixed">
+    <parent link="base_link"/>
+    <child link="chassis"/>
+    <origin xyz="0 0 0"/>
+  </joint>
+  <link name="chassis">
     <visual>
       <geometry>
@@ -28,7 +36,14 @@
     </inertial>
   </link>
-<gazebo reference="base_link">
+<gazebo reference="chassis">
     <material>Gazebo/White</material>
 </gazebo>
+<!-- BASE_FOOTPRINT LINK
+<joint name="base_footprint_joint" type="fixed">
+  <parent link="base_link"/>
+  <child link="base_footprint"/>
+  <origin xyz ="0 0 0" rpy="0 0 0"/>
+</joint>
+ -->
   <!-- Controlled Wheels -->
   <xacro:macro name="wheel" params="name x y w">
