Commit message: redesigned robot similar to a roomba

File: src/mollyBot/description/robot_core.xacro (robot description, xacro)
@@ -70,5 +70,5 @@
     <inertial>
       <origin xyz="0 0 0"/>
-      <mass value="0.5"/>
+      <mass value="0.3"/>
       <inertia ixx="0.0001" ixy="0.0" ixz="0.0" iyy="0.0001" iyz="0.0" izz="0.0001"/>
     </inertial>
@@ -82,5 +82,5 @@
     <parent link="base_link"/>
     <child link="caster_wheel"/>
-    <origin xyz="0.2 0 -0.03" rpy="0 0 0"/>
+    <origin xyz="0.2 0 -0.05" rpy="0 0 0"/>
   </joint>
 </robot>

Commit message: Added SLAM config files and saved a SLAM map of blockroom.world

File: src/mollyBot/description/robot_core.xacro (robot description, xacro)
@@ -13,4 +13,12 @@
   <link name="base_link">
   </link>
+<!-- BASE_FOOTPRINT LINK -->
+<joint name="base_footprint_joint" type="fixed">
+  <parent link="base_link"/>
+  <child link="base_footprint"/>
+  <origin xyz ="0 0 0" rpy="0 0 0"/>
+</joint>
+<link name="base_footprint">
+</link>
   <!-- Chassis Link -->
   <joint name="chassis_joint" type="fixed">
@@ -39,11 +47,4 @@
     <material>Gazebo/White</material>
 </gazebo>
-<!-- BASE_FOOTPRINT LINK
-<joint name="base_footprint_joint" type="fixed">
-  <parent link="base_link"/>
-  <child link="base_footprint"/>
-  <origin xyz ="0 0 0" rpy="0 0 0"/>
-</joint>
- -->
   <!-- Controlled Wheels -->
   <xacro:macro name="wheel" params="name x y w">
